File: hardware/main-board/ESP32.sch (KiCad schematic (older format))
At the start: 8 parts

Commit message: Added USB to uart
Parts:
- added C?: 0.1uF, symbol Device:C_Small
- added C?: 10uF, symbol Device:C_Small
- added R?: 2k, symbol Device:R_US
- added R?: 22.1k, symbol Device:R_US
- added R?: 47.5k, symbol Device:R_US
Connections:
- wire segments 46 -> 70
- no-connect marks 2 -> 18
Other:
- moved on the sheet: C?, U?
