File: hardware/main-board/ESP32.sch (KiCad schematic (older format))
At the start: 19 parts

Commit message: Sch mostly done, drew a few custom footprints, placement mostly done.
Parts:
- removed D?: D, symbol Device:D
- removed D?: CM1293A-04SO, Package_TO_SOT_SMD:SOT-23-6, symbol main-board-custom-symbols:CM1293A-04SO
- removed J?: USB-C Receptacle, symbol Connector:USB_C_Receptacle_USB2.0
- removed R? (x2): 5.1k, symbol Device:R_US
- added C7: 0.1uF, Capacitor_SMD:C_0603_1608Metric, symbol Device:C_Small
- added JP1: EN jumper, Jumper:SolderJumper-2_P1.3mm_Open_RoundedPad1.0x1.5mm, symbol Jumper:Jumper_2_Open
- added JP2: BOOT jumper, Jumper:SolderJumper-2_P1.3mm_Open_RoundedPad1.0x1.5mm, symbol Jumper:Jumper_2_Open
- C4, C8: renamed from C?; footprint (none) -> Capacitor_SMD:C_0805_2012Metric
- C5, C6: renamed from C?; footprint (none) -> Capacitor_SMD:C_0603_1608Metric
- Q2, Q3: renamed from Q?; footprint (none) -> Package_TO_SOT_SMD:SOT-23
- R10, R11, R12, R13, R14, R9: renamed from R?; footprint (none) -> Resistor_SMD:R_0603_1608Metric
- U4: renamed from U?; MPN (none) -> CP2102N-A01-GQFN28
- U5: renamed from U?; MPN (none) -> ESP32-WROOM-32
Connections:
- net labels added: CANBUS_RX, CANBUS_TERM_EN, CANBUS_TX, FRONT_BUTTON, LCD_BACKLIGHT, LCD_CS, LCD_DC, LCD_RESET, LCD_SCL, LCD_SDO, PROG_RX, PROG_TXD
- net labels removed: +5V, RXD, TXD, USB_CC1, USB_CC2
- wire segments 94 -> 69
Other:
- moved on the sheet: C4, C5, C8, Q2, Q3, R10, R11, R12, R13, R9, U4

Commit message: layout almost done
Connections:
- net CANBUS_TERM_EN: now also U5.24 (IO2)
Changed lines of the file:
@@
 EESchema Schematic File Version 4
-LIBS:main-board-cache
-EELAYER 29 0
+EELAYER 30 0
 EELAYER END
 $Descr B 17000 11000
@@
 Wire Wire Line
 	12800 6250 12700 6250
-Text HLabel 13800 5250 2    50   Output ~ 0
+Text HLabel 12800 4550 2    50   Output ~ 0
 CANBUS_TERM_EN
 Text HLabel 2550 4000 0    50   Input ~ 0
@@
 Wire Wire Line
 	3600 5050 2550 5050
+Wire Wire Line
+	12700 4550 12800 4550
 $EndSCHEMATC

Commit message: BOM cleanup/adding MPNs
Parts:
- C4, C8: MPN (none) -> CL21B106KQQNFNE
- C5, C6, C7: MPN (none) -> CL10B104KA8NFNC
- R10: value 47.5k -> 10k; MPN (none) -> RC0603JR-0710KL
- R11: value 2k -> 5.1k; MPN (none) -> RC0603JR-075K1L
- R12, R13, R14: MPN (none) -> RC0603JR-0710KL
- R9: value 22.1k -> 5.1k; MPN (none) -> RC0603JR-075K1L
Changed lines of the file:
@@
 F 2 "Capacitor_SMD:C_0805_2012Metric" H 11750 3850 50  0001 C CNN
 F 3 "~" H 11750 3850 50  0001 C CNN
+F 4 "CL21B106KQQNFNE" H 11750 3850 50  0001 C CNN "MPN"
 	1    11750 3850
 	1    0    0    -1
@@
 F 2 "Capacitor_SMD:C_0603_1608Metric" H 4350 3600 50  0001 C CNN
 F 3 "~" H 4350 3600 50  0001 C CNN
+F 4 "CL10B104KA8NFNC" H 4350 3600 50  0001 C CNN "MPN"
 	1    4350 3600
 	1    0    0    -1
@@
 F 2 "Capacitor_SMD:C_0805_2012Metric" H 3950 3600 50  0001 C CNN
 F 3 "~" H 3950 3600 50  0001 C CNN
+F 4 "CL21B106KQQNFNE" H 3950 3600 50  0001 C CNN "MPN"
 	1    3950 3600
 	1    0    0    -1
@@
 P 4100 4250
 F 0 "R11" V 3895 4250 50  0000 C CNN
-F 1 "2k" V 3986 4250 50  0000 C CNN
+F 1 "5.1k" V 3986 4250 50  0000 C CNN
 F 2 "Resistor_SMD:R_0603_1608Metric" V 4140 4240 50  0001 C CNN
 F 3 "~" H 4100 4250 50  0001 C CNN
+F 4 "RC0603JR-075K1L" H 4100 4250 50  0001 C CNN "MPN"
 	1    4100 4250
 	0    1    1    0
@@
 P 3000 4150
 F 0 "R9" H 2932 4104 50  0000 R CNN
-F 1 "22.1k" H 2932 4195 50  0000 R CNN
+F 1 "5.1k" H 2932 4195 50  0000 R CNN
 F 2 "Resistor_SMD:R_0603_1608Metric" V 3040 4140 50  0001 C CNN
 F 3 "~" H 3000 4150 50  0001 C CNN
+F 4 "RC0603JR-075K1L" H 3000 4150 50  0001 C CNN "MPN"
 	1    3000 4150
 	-1   0    0    1
@@
 P 3000 4450
 F 0 "R10" H 2932 4404 50  0000 R CNN
-F 1 "47.5k" H 2932 4495 50  0000 R CNN
+F 1 "10k" H 2932 4495 50  0000 R CNN
 F 2 "Resistor_SMD:R_0603_1608Metric" V 3040 4440 50  0001 C CNN
 F 3 "~" H 3000 4450 50  0001 C CNN
+F 4 "RC0603JR-0710KL" H 3000 4450 50  0001 C CNN "MPN"
 	1    3000 4450
 	-1   0    0    1
@@
 F 2 "Resistor_SMD:R_0603_1608Metric" V 6240 5240 50  0001 C CNN
 F 3 "~" H 6200 5250 50  0001 C CNN
+F 4 "RC0603JR-0710KL" H 6200 5250 50  0001 C CNN "MPN"
 	1    6200 5250
 	0    1    1    0
@@
 F 2 "Resistor_SMD:R_0603_1608Metric" V 6240 5940 50  0001 C CNN
 F 3 "~" H 6200 5950 50  0001 C CNN
+F 4 "RC0603JR-0710KL" H 6200 5950 50  0001 C CNN "MPN"
 	1    6200 5950
 	0    1    1    0
@@
 F 2 "Resistor_SMD:R_0603_1608Metric" V 10940 4140 50  0001 C CNN
 F 3 "~" H 10900 4150 50  0001 C CNN
+F 4 "RC0603JR-0710KL" H 10900 4150 50  0001 C CNN "MPN"
 	1    10900 4150
 	1    0    0    -1
@@
 F 2 "Capacitor_SMD:C_0603_1608Metric" H 10900 4500 50  0001 C CNN
 F 3 "~" H 10900 4500 50  0001 C CNN
+F 4 "CL10B104KA8NFNC" H 10900 4500 50  0001 C CNN "MPN"
 	1    10900 4500
 	1    0    0    -1
@@
 F 2 "Capacitor_SMD:C_0603_1608Metric" H 11350 3850 50  0001 C CNN
 F 3 "~" H 11350 3850 50  0001 C CNN
+F 4 "CL10B104KA8NFNC" H 11350 3850 50  0001 C CNN "MPN"
 	1    11350 3850
 	1    0    0    -1

Commit message: further BOM fixing/cleanup for ordering.
Parts:
- U5: MPN ESP32-WROOM-32 -> ESP32-WROOM-32D
Changed lines of the file:
@@
 F 2 "RF_Module:ESP32-WROOM-32" H 12100 4050 50  0001 C CNN
 F 3 "https://www.espressif.com/sites/default/files/documentation/esp32-wroom-32_datasheet_en.pdf" H 11800 5600 50  0001 C CNN
-F 4 "ESP32-WROOM-32" H 12100 5550 50  0001 C CNN "MPN"
+F 4 "ESP32-WROOM-32D" H 12100 5550 50  0001 C CNN "MPN"
 	1    12100 5550
 	1    0    0    -1
