File: hardware/main-board/CANbus.sch (KiCad schematic (older format))
At the start: 0 parts

Commit message: Sch mostly done, drew a few custom footprints, placement mostly done.
Parts:
- added C1: 0.1uF, Capacitor_SMD:C_0603_1608Metric, symbol Device:C_Small
- added D5: NUP2105L, Package_TO_SOT_SMD:SOT-23, symbol Power_Protection:NUP2105L
- added FL1: EMI_Filter_CommonMode, main-board-custom-footprints:COMMON_MODE_CHOKE_BOURNS_DR331, symbol Device:EMI_Filter_LL_1423
- added R3: 10k, Resistor_SMD:R_0603_1608Metric, symbol Device:R_US
- added R4: 400R, Resistor_SMD:R_0603_1608Metric, symbol Device:R_US
- added R5: 120R, Resistor_SMD:R_0603_1608Metric, symbol Device:R_US
- added U1: SN65HVD230, Package_SO:SOIC-8_3.9x4.9mm_P1.27mm, symbol Interface_CAN_LIN:SN65HVD230
- added U2: CPC1017N, Package_SO:SOP-4_3.8x4.1mm_P2.54mm, symbol Relay_SolidState:CPC1017N
Connections:
- new net: D5.1 (K), FL1.1, U1.6 (CANL)
- new net: D5.2 (K), FL1.2, U1.7 (CANH)
- new net: R3.1, U1.8 (Rs)
- new net: R4.1, U2.1
- new net: R5.2, U2.3
- new net +3V3: C1.1, U1.3 (VCC)
- new net CANH: FL1.3, R5.1
- new net CANL: FL1.4, U2.4
- new net CAN_RX: U1.4 (R)
- new net CAN_TERM_EN: R4.2
- new net CAN_TX: U1.1 (D)
- new net GND: C1.2, D5.3 (A), R3.2, U1.2 (GND), U2.2
- no-connect marks 0 -> 1
Other:
- note added: "Software-controlled termination"
