File: hardware/main-board/CANbus.sch (KiCad schematic (older format))
At the start: 8 parts, among them U1 SN65HVD230, U2 CPC1017N

Commit message: added qr code, switched button to a different button. put on reddit for review
Parts:
- FL1: value EMI_Filter_CommonMode -> DR331-513AE
Changed lines of the file:
@@
 EESchema Schematic File Version 4
-LIBS:main-board-cache
-EELAYER 29 0
+EELAYER 30 0
 EELAYER END
 $Descr B 17000 11000
@@
 P 10150 5200
 F 0 "FL1" H 10150 5481 50  0000 C CNN
-F 1 "EMI_Filter_CommonMode" H 10150 5390 50  0000 C CNN
+F 1 "DR331-513AE" H 10150 5390 50  0000 C CNN
 F 2 "main-board-custom-footprints:COMMON_MODE_CHOKE_BOURNS_DR331" H 10150 5240 50  0001 C CNN
 F 3 "~" H 10150 5240 50  0001 C CNN

Commit message: Added mounting holes, tweaked layout to accomodate.
Connections:
- net at FL1.1, U1.6 (CANL): now also D5.2 (K); no longer D5.1 (K)
- net at FL1.2, U1.7 (CANH): now also D5.1 (K); no longer D5.2 (K)
Changed lines of the file:
@@
 EESchema Schematic File Version 4
-EELAYER 30 0
+LIBS:main-board-cache
+EELAYER 29 0
 EELAYER END
 $Descr B 17000 11000
@@
 Wire Wire Line
 	10400 5300 10400 5250
-Wire Wire Line
-	9300 5350 9300 5250
-Wire Wire Line
-	9500 5350 9500 5150
 $Comp
 L power:GND #PWR015
@@
 	10400 5250 10800 5250
 Wire Wire Line
-	9000 5250 9300 5250
-Connection ~ 9300 5250
-Wire Wire Line
-	9000 5150 9500 5150
-Connection ~ 9500 5150
-Wire Wire Line
 	10350 5300 10400 5300
 Wire Wire Line
@@
 	9900 5100 9950 5100
 Wire Wire Line
-	9500 5150 9900 5150
-Wire Wire Line
 	9900 5250 9900 5300
 Wire Wire Line
 	9900 5300 9950 5300
-Wire Wire Line
-	9300 5250 9900 5250
 Wire Wire Line
 	10800 5650 10800 5250
@@
 	1    0    0    -1
 $EndComp
+Wire Wire Line
+	9000 5250 9500 5250
+Wire Wire Line
+	9000 5150 9300 5150
+Wire Wire Line
+	9500 5350 9500 5250
+Connection ~ 9500 5250
+Wire Wire Line
+	9500 5250 9900 5250
+Wire Wire Line
+	9300 5350 9300 5150
+Connection ~ 9300 5150
+Wire Wire Line
+	9300 5150 9900 5150
 $EndSCHEMATC

Commit message: BOM cleanup/adding MPNs
Parts:
- C1: MPN (none) -> CL10B104KA8NFNC
- R3: MPN (none) -> RC0603JR-0710KL
- R4: value 400R -> 470R; MPN (none) -> RC0603JR-07470RL
- R5: value 120R -> 100R; MPN (none) -> RC0603JR-07100RL
Changed lines of the file:
@@
 F 2 "Resistor_SMD:R_0603_1608Metric" V 8090 5590 50  0001 C CNN
 F 3 "~" H 8050 5600 50  0001 C CNN
+F 4 "RC0603JR-0710KL" H 8050 5600 50  0001 C CNN "MPN"
 	1    8050 5600
 	1    0    0    -1
@@
 F 2 "Capacitor_SMD:C_0603_1608Metric" H 8000 4550 50  0001 C CNN
 F 3 "~" H 8000 4550 50  0001 C CNN
+F 4 "CL10B104KA8NFNC" H 8000 4550 50  0001 C CNN "MPN"
 	1    8000 4550
 	1    0    0    -1
@@
 P 11000 5500
 F 0 "R5" H 11068 5546 50  0000 L CNN
-F 1 "120R" H 11068 5455 50  0000 L CNN
+F 1 "100R" H 11068 5455 50  0000 L CNN
 F 2 "Resistor_SMD:R_0603_1608Metric" V 11040 5490 50  0001 C CNN
 F 3 "~" H 11000 5500 50  0001 C CNN
+F 4 "RC0603JR-07100RL" H 11000 5500 50  0001 C CNN "MPN"
 	1    11000 5500
 	1    0    0    -1
@@
 P 10550 6400
 F 0 "R4" V 10345 6400 50  0000 C CNN
-F 1 "400R" V 10436 6400 50  0000 C CNN
+F 1 "470R" V 10436 6400 50  0000 C CNN
 F 2 "Resistor_SMD:R_0603_1608Metric" V 10590 6390 50  0001 C CNN
 F 3 "~" H 10550 6400 50  0001 C CNN
+F 4 "RC0603JR-07470RL" H 10550 6400 50  0001 C CNN "MPN"
 	1    10550 6400
 	0    1    1    0

Commit message: further BOM fixing/cleanup for ordering.
Parts:
- D5: MPN NUP2105L -> NUP2105LT1G
Changed lines of the file:
@@
 F 2 "Package_TO_SOT_SMD:SOT-23" H 9625 5500 50  0001 L CNN
 F 3 "http://www.onsemi.com/pub_link/Collateral/NUP2105L-D.PDF" H 9525 5675 50  0001 C CNN
-F 4 "NUP2105L" H 9400 5550 50  0001 C CNN "MPN"
+F 4 "NUP2105LT1G" H 9400 5550 50  0001 C CNN "MPN"
 	1    9400 5550
 	1    0    0    -1
