File: hardware/main-board/LCD.sch (KiCad schematic (older format))
At the start: 0 parts

Commit message: Sch mostly done, drew a few custom footprints, placement mostly done.
Parts:
- added J3: LCD_FFC_SOLDER, main-board-custom-footprints:LCD_ROUND_IPS_ER-TFT1.28-1, symbol Connector_Generic:Conn_01x12
- added Q1: SS8050-G, Package_TO_SOT_SMD:SOT-23, symbol Device:Q_NPN_BEC
- added R6: 1k, Resistor_SMD:R_0603_1608Metric, symbol Device:R_US
- added R7: 10k, Resistor_SMD:R_0603_1608Metric, symbol Device:R_US
- added R8: 10R, Resistor_SMD:R_0603_1608Metric, symbol Device:R_US
Connections:
- new net: J3.2 (Pin_2), R8.1
- new net: Q1.1 (B), R6.1, R7.1
- new net: Q1.3 (C), R8.2
- new net +3V3: J3.3 (Pin_3), J3.4 (Pin_4), R7.2
- new net BACKLIGHT: R6.2
- new net CS: J3.8 (Pin_8)
- new net DC: J3.7 (Pin_7)
- new net GND: J3.1 (Pin_1), J3.12 (Pin_12), J3.5 (Pin_5), J3.6 (Pin_6), Q1.2 (E)
- new net RST: J3.11 (Pin_11)
- new net SCL: J3.9 (Pin_9)
- new net SDI: J3.10 (Pin_10)
Changed lines of the file:
@@
 EESchema Schematic File Version 4
-EELAYER 30 0
+LIBS:main-board-cache
+EELAYER 29 0
 EELAYER END
-$Descr A4 11693 8268
+$Descr B 17000 11000
 encoding utf-8
-Sheet 1 5
+Sheet 4 5
 Title ""
 Date ""
@@
 Comment4 ""
 $EndDescr
+$Comp
+L Connector_Generic:Conn_01x12 J3
+U 1 1 610023D7
+P 9700 4800
+F 0 "J3" H 9780 4792 50  0000 L CNN
+F 1 "LCD_FFC_SOLDER" H 9780 4701 50  0000 L CNN
+F 2 "main-board-custom-footprints:LCD_ROUND_IPS_ER-TFT1.28-1" H 9700 4800 50  0001 C CNN
+F 3 "~" H 9700 4800 50  0001 C CNN
+F 4 "DNP" H 9700 4800 50  0001 C CNN "MPN"
+	1    9700 4800
+	1    0    0    -1
+$EndComp
+Wire Wire Line
+	9400 4300 9500 4300
+$Comp
+L power:GND #PWR024
+U 1 1 61003347
+P 9400 4300
+F 0 "#PWR024" H 9400 4050 50  0001 C CNN
+F 1 "GND" V 9405 4172 50  0000 R CNN
+F 2 "" H 9400 4300 50  0001 C CNN
+F 3 "" H 9400 4300 50  0001 C CNN
+	1    9400 4300
+	0    1    1    0
+$EndComp
+$Comp
+L power:GND #PWR026
+U 1 1 61005807
+P 9400 4750
+F 0 "#PWR026" H 9400 4500 50  0001 C CNN
+F 1 "GND" V 9405 4622 50  0000 R CNN
+F 2 "" H 9400 4750 50  0001 C CNN
+F 3 "" H 9400 4750 50  0001 C CNN
+	1    9400 4750
+	0    1    1    0
+$EndComp
+Wire Wire Line
+	9400 5400 9500 5400
+$Comp
+L power:GND #PWR027
+U 1 1 61005A4E
+P 9400 5400
+F 0 "#PWR027" H 9400 5150 50  0001 C CNN
+F 1 "GND" V 9405 5272 50  0000 R CNN
+F 2 "" H 9400 5400 50  0001 C CNN
+F 3 "" H 9400 5400 50  0001 C CNN
+	1    9400 5400
+	0    1    1    0
+$EndComp
+Wire Wire Line
+	9500 4700 9450 4700
+Wire Wire Line
+	9450 4700 9450 4750
+Wire Wire Line
+	9450 4800 9500 4800
+Wire Wire Line
+	9400 4750 9450 4750
+Connection ~ 9450 4750
+Wire Wire Line
+	9450 4750 9450 4800
+$Comp
+L Device:Q_NPN_BEC Q?
+U 1 1 61008515
+P 8350 4600
+AR Path="/60F6511D/61008515" Ref="Q?"  Part="1"
+AR Path="/60F65232/61008515" Ref="Q1"  Part="1"
+F 0 "Q1" H 8540 4646 50  0000 L CNN
+F 1 "SS8050-G" H 8540 4555 50  0000 L CNN
+F 2 "Package_TO_SOT_SMD:SOT-23" H 8550 4700 50  0001 C CNN
+F 3 "~" H 8350 4600 50  0001 C CNN
+F 4 "SS8050-G" H 8350 4600 50  0001 C CNN "MPN"
+	1    8350 4600
+	1    0    0    -1
+$EndComp
+$Comp
+L Device:R_US R8
+U 1 1 61009737
+P 8800 4300
+F 0 "R8" V 8595 4300 50  0000 C CNN
+F 1 "10R" V 8686 4300 50  0000 C CNN
+F 2 "Resistor_SMD:R_0603_1608Metric" V 8840 4290 50  0001 C CNN
+F 3 "~" H 8800 4300 50  0001 C CNN
+	1    8800 4300
+	0    1    1    0
+$EndComp
+$Comp
+L Device:R_US R6
+U 1 1 6100BCFB
+P 7750 4600
+F 0 "R6" V 7545 4600 50  0000 C CNN
+F 1 "1k" V 7636 4600 50  0000 C CNN
+F 2 "Resistor_SMD:R_0603_1608Metric" V 7790 4590 50  0001 C CNN
+F 3 "~" H 7750 4600 50  0001 C CNN
+	1    7750 4600
+	0    1    1    0
+$EndComp
+$Comp
+L Device:R_US R7
+U 1 1 6100C16B
+P 8050 4350
+F 0 "R7" H 7982 4304 50  0000 R CNN
+F 1 "10k" H 7982 4395 50  0000 R CNN
+F 2 "Resistor_SMD:R_0603_1608Metric" V 8090 4340 50  0001 C CNN
+F 3 "~" H 8050 4350 50  0001 C CNN
+	1    8050 4350
+	-1   0    0    1
+$EndComp
+$Comp
+L power:+3.3V #PWR022
+U 1 1 6100D0C9
+P 8050 4200
+F 0 "#PWR022" H 8050 4050 50  0001 C CNN
+F 1 "+3.3V" H 8065 4373 50  0000 C CNN
+F 2 "" H 8050 4200 50  0001 C CNN
+F 3 "" H 8050 4200 50  0001 C CNN
+	1    8050 4200
+	1    0    0    -1
+$EndComp
+Wire Wire Line
+	8150 4600 8050 4600
+Wire Wire Line
+	8050 4600 8050 4500
+Wire Wire Line
+	7900 4600 8050 4600
+Connection ~ 8050 4600
+Wire Wire Line
+	9500 4400 9050 4400
+Wire Wire Line
+	9050 4400 9050 4300
+Wire Wire Line
+	9050 4300 8950 4300
+Wire Wire Line
+	8650 4300 8450 4300
+Wire Wire Line
+	8450 4300 8450 4400
+$Comp
+L power:+3.3V #PWR025
+U 1 1 61013AAE
+P 9400 4550
+F 0 "#PWR025" H 9400 4400 50  0001 C CNN
+F 1 "+3.3V" V 9415 4678 50  0000 L CNN
+F 2 "" H 9400 4550 50  0001 C CNN
+F 3 "" H 9400 4550 50  0001 C CNN
+	1    9400 4550
+	0    -1   -1   0
+$EndComp
+Wire Wire Line
+	9500 4500 9450 4500
+Wire Wire Line
+	9450 4500 9450 4550
+Wire Wire Line
+	9450 4600 9500 4600
+Wire Wire Line
+	9400 4550 9450 4550
+Connection ~ 9450 4550
+Wire Wire Line
+	9450 4550 9450 4600
+Wire Wire Line
+	9500 4900 8950 4900
+Wire Wire Line
+	9500 5000 8950 5000
+Wire Wire Line
+	9500 5100 8950 5100
+Wire Wire Line
+	9500 5200 8950 5200
+Wire Wire Line
+	9500 5300 8950 5300
+Text HLabel 8950 4900 0    50   Input ~ 0
+DC
+Text HLabel 8950 5000 0    50   Input ~ 0
+CS
+Text HLabel 8950 5100 0    50   Input ~ 0
+SCL
+Text HLabel 8950 5200 0    50   Input ~ 0
+SDI
+Text HLabel 8950 5300 0    50   Input ~ 0
+RST
+$Comp
+L power:GND #PWR023
+U 1 1 61020E01
+P 8450 4800
+F 0 "#PWR023" H 8450 4550 50  0001 C CNN
+F 1 "GND" H 8455 4627 50  0000 C CNN
+F 2 "" H 8450 4800 50  0001 C CNN
+F 3 "" H 8450 4800 50  0001 C CNN
+	1    8450 4800
+	1    0    0    -1
+$EndComp
+Text HLabel 7600 4600 0    50   Input ~ 0
+BACKLIGHT
 $EndSCHEMATC
