File: hardware/main-board/LCD.sch (KiCad schematic (older format))
At the start: 5 parts, among them J3 LCD_FFC_SOLDER, Q1 SS8050-G

Commit message: BOM cleanup/adding MPNs
Parts:
- R6: value 1k -> 470R; MPN (none) -> RC0603JR-07470RL
- R7: MPN (none) -> RC0603JR-0710KL
- R8: MPN (none) -> RC0603JR-0710RL
Changed lines of the file:
@@
 F 2 "Resistor_SMD:R_0603_1608Metric" V 8840 4290 50  0001 C CNN
 F 3 "~" H 8800 4300 50  0001 C CNN
+F 4 "RC0603JR-0710RL" H 8800 4300 50  0001 C CNN "MPN"
 	1    8800 4300
 	0    1    1    0
@@
 P 7750 4600
 F 0 "R6" V 7545 4600 50  0000 C CNN
-F 1 "1k" V 7636 4600 50  0000 C CNN
+F 1 "470R" V 7636 4600 50  0000 C CNN
 F 2 "Resistor_SMD:R_0603_1608Metric" V 7790 4590 50  0001 C CNN
 F 3 "~" H 7750 4600 50  0001 C CNN
+F 4 "RC0603JR-07470RL" H 7750 4600 50  0001 C CNN "MPN"
 	1    7750 4600
 	0    1    1    0
@@
 F 2 "Resistor_SMD:R_0603_1608Metric" V 8090 4340 50  0001 C CNN
 F 3 "~" H 8050 4350 50  0001 C CNN
+F 4 "RC0603JR-0710KL" H 8050 4350 50  0001 C CNN "MPN"
 	1    8050 4350
 	-1   0    0    1
