File: hardware/main-board/PSU.sch (KiCad schematic (older format))
At the start: 0 parts

Commit message: Sch mostly done, drew a few custom footprints, placement mostly done.
Parts:
- added C2: 10uF, Capacitor_SMD:C_1210_3225Metric, symbol Device:C_Small
- added C3: 10uF, Capacitor_SMD:C_0805_2012Metric, symbol Device:C_Small
- added D6: 30V 1A, Diode_SMD:D_SMA, symbol Device:D_Schottky
- added L1: 47uH, Inductor_SMD:L_Taiyo-Yuden_NR-60xx, symbol Device:L
- added U3: AP1509-33SG-13, Package_SO:SO-8_3.9x4.9mm_P1.27mm, symbol main-board-custom-symbols:AP1509-50
Connections:
- new net: D6.1 (K), L1.1, U3.2 (OUTPUT)
- new net 3.3VOUT: C3.1, L1.2
- new net GND: C2.2, C3.2, D6.2 (A), U3.4 (SD), U3.5 (GND), U3.6 (GND), U3.7 (GND), U3.8 (GND)
- new net VIN: C2.1, U3.1 (VIN)
- no-connect marks 0 -> 1
Changed lines of the file:
@@
 EESchema Schematic File Version 4
-EELAYER 30 0
+LIBS:main-board-cache
+EELAYER 29 0
 EELAYER END
-$Descr A4 11693 8268
+$Descr B 17000 11000
 encoding utf-8
-Sheet 1 5
+Sheet 3 5
 Title ""
 Date ""
@@
 Comment4 ""
 $EndDescr
+$Comp
+L main-board-custom-symbols:AP1509-50 U3
+U 1 1 60FCBB15
+P 5800 5150
+F 0 "U3" H 5800 5565 50  0000 C CNN
+F 1 "AP1509-33SG-13" H 5800 5474 50  0000 C CNN
+F 2 "Package_SO:SO-8_3.9x4.9mm_P1.27mm" H 5750 5250 50  0001 C CNN
+F 3 "" H 5750 5250 50  0001 C CNN
+F 4 "AP1509-33SG-13" H 5800 5150 50  0001 C CNN "MPN"
+	1    5800 5150
+	1    0    0    -1
+$EndComp
+NoConn ~ 6200 5200
+Wire Wire Line
+	5400 5200 5300 5200
+$Comp
+L power:GND #PWR019
+U 1 1 60FCC50A
+P 5800 5500
+F 0 "#PWR019" H 5800 5250 50  0001 C CNN
+F 1 "GND" H 5805 5327 50  0000 C CNN
+F 2 "" H 5800 5500 50  0001 C CNN
+F 3 "" H 5800 5500 50  0001 C CNN
+	1    5800 5500
+	1    0    0    -1
+$EndComp
+$Comp
+L power:GND #PWR018
+U 1 1 60FCC70B
+P 5300 5500
+F 0 "#PWR018" H 5300 5250 50  0001 C CNN
+F 1 "GND" H 5305 5327 50  0000 C CNN
+F 2 "" H 5300 5500 50  0001 C CNN
+F 3 "" H 5300 5500 50  0001 C CNN
+	1    5300 5500
+	1    0    0    -1
+$EndComp
+Wire Wire Line
+	5300 5200 5300 5500
+$Comp
+L Device:C_Small C2
+U 1 1 60FCCE2C
+P 4850 5250
+F 0 "C2" H 4942 5296 50  0000 L CNN
+F 1 "10uF" H 4942 5205 50  0000 L CNN
+F 2 "Capacitor_SMD:C_1210_3225Metric" H 4850 5250 50  0001 C CNN
+F 3 "~" H 4850 5250 50  0001 C CNN
+	1    4850 5250
+	1    0    0    -1
+$EndComp
+Wire Wire Line
+	5400 5000 4850 5000
+Wire Wire Line
+	4850 5000 4850 5150
+$Comp
+L power:GND #PWR017
+U 1 1 60FCD6A2
+P 4850 5500
+F 0 "#PWR017" H 4850 5250 50  0001 C CNN
+F 1 "GND" H 4855 5327 50  0000 C CNN
+F 2 "" H 4850 5500 50  0001 C CNN
+F 3 "" H 4850 5500 50  0001 C CNN
+	1    4850 5500
+	1    0    0    -1
+$EndComp
+Wire Wire Line
+	4850 5350 4850 5500
+$Comp
+L Device:D_Schottky D6
+U 1 1 60FCE5F1
+P 6550 5300
+F 0 "D6" V 6504 5379 50  0000 L CNN
+F 1 "30V 1A" V 6595 5379 50  0000 L CNN
+F 2 "Diode_SMD:D_SMA" H 6550 5300 50  0001 C CNN
+F 3 "~" H 6550 5300 50  0001 C CNN
+F 4 "SS13MHRSG" V 6550 5300 50  0001 C CNN "MPN"
+	1    6550 5300
+	0    1    1    0
+$EndComp
+$Comp
+L power:GND #PWR020
+U 1 1 60FCEC10
+P 6550 5500
+F 0 "#PWR020" H 6550 5250 50  0001 C CNN
+F 1 "GND" H 6555 5327 50  0000 C CNN
+F 2 "" H 6550 5500 50  0001 C CNN
+F 3 "" H 6550 5500 50  0001 C CNN
+	1    6550 5500
+	1    0    0    -1
+$EndComp
+Wire Wire Line
+	6550 5450 6550 5500
+Wire Wire Line
+	6200 5000 6550 5000
+Wire Wire Line
+	6550 5000 6550 5150
+$Comp
+L Device:L L1
+U 1 1 60FCF9E1
+P 6850 5000
+F 0 "L1" V 7040 5000 50  0000 C CNN
+F 1 "47uH" V 6949 5000 50  0000 C CNN
+F 2 "Inductor_SMD:L_Taiyo-Yuden_NR-60xx" H 6850 5000 50  0001 C CNN
+F 3 "~" H 6850 5000 50  0001 C CNN
+F 4 "NRS6045T470MMGKV" V 6850 5000 50  0001 C CNN "MPN"
+	1    6850 5000
+	0    -1   -1   0
+$EndComp
+Wire Wire Line
+	6550 5000 6700 5000
+Connection ~ 6550 5000
+$Comp
+L Device:C_Small C3
+U 1 1 60FCFF6B
+P 7200 5250
+F 0 "C3" H 7292 5296 50  0000 L CNN
+F 1 "10uF" H 7292 5205 50  0000 L CNN
+F 2 "Capacitor_SMD:C_0805_2012Metric" H 7200 5250 50  0001 C CNN
+F 3 "~" H 7200 5250 50  0001 C CNN
+	1    7200 5250
+	1    0    0    -1
+$EndComp
+Wire Wire Line
+	7000 5000 7200 5000
+Wire Wire Line
+	7200 5000 7200 5150
+$Comp
+L power:GND #PWR021
+U 1 1 60FD0BAC
+P 7200 5500
+F 0 "#PWR021" H 7200 5250 50  0001 C CNN
+F 1 "GND" H 7205 5327 50  0000 C CNN
+F 2 "" H 7200 5500 50  0001 C CNN
+F 3 "" H 7200 5500 50  0001 C CNN
+	1    7200 5500
+	1    0    0    -1
+$EndComp
+Wire Wire Line
+	7200 5350 7200 5500
+Text HLabel 4700 5000 0    50   Input ~ 0
+VIN
+Wire Wire Line
+	7200 5000 7550 5000
+Connection ~ 7200 5000
+Text HLabel 7550 5000 2    50   Output ~ 0
+3.3VOUT
+Wire Wire Line
+	4700 5000 4850 5000
+Connection ~ 4850 5000
 $EndSCHEMATC
