File: hardware/main-board/main-board.sch (KiCad schematic (older format))
At the start: 14 parts, among them J1 USB-C Receptacle, J2 JST JWPF, SW1 FRONT_BUTTON

Commit message: cleaning up BOM
Parts:
- SW1: MPN B3S-1100P -> PTS810 SJG 250 SMTR LFS
Changed lines of the file:
@@
 F 2 "main-board-custom-footprints:SW_SPST_PTS810" H 11500 5600 50  0001 C CNN
 F 3 "~" H 11500 5600 50  0001 C CNN
-F 4 "B3S-1100P" H 11500 5400 50  0001 C CNN "MPN"
+F 4 "PTS810 SJG 250 SMTR LFS" H 11500 5400 50  0001 C CNN "MPN"
 	1    11500 5400
 	1    0    0    -1
